File: Hardware/socket/in14-socket/in14-socket.sch (KiCad schematic (older format))
At the start: 1 part

Commit message: logic PCB tweaks, resize
Parts:
- added GL1: NE2-NEON-BULB-DRILL, mynixies:mynixies-NE2-NEON-BULB-DRILL, symbol mynixies:NE2-NEON-BULB-DRILL
- added J3: Conn_01x20_Male, Connector_IDC:IDC-Header_2x10_P2.54mm_Horizontal, symbol Connector:Conn_01x20_Male
- added LED1, LED2, LED3, LED4: VLMU3100-GS08, footprints:VLMU3100-GS08, symbol VLMU3100-GS08:VLMU3100-GS08
- added N2, N3, N4: IN-14, nixies-us:nixies-us-IN-14, symbol nixies-us:IN-14
- added Q1, Q2: BC847BS, Package_TO_SOT_SMD:SOT-363_SC-70-6, symbol Transistor_BJT:BC847BS
- added RA9: 220 x 4, Resistor_SMD:R_Array_Convex_4x0603, symbol Device:R_Pack04
- added RV1: R_POT_TRIM_US, footprints:TRIM_3362P-1-302LF, symbol Device:R_POT_TRIM_US
- N1: renamed from N?; footprint nixies-us_IN-14 -> nixies-us:nixies-us-IN-14
Connections:
- net at N1.0: now also J3.9 (Pin_9), N2.0, N3.0, N4.0
- net at N1.1: now also J3.10 (Pin_10), N2.1, N3.1, N4.1
- net at N1.2: now also J3.11 (Pin_11), N2.2, N3.2, N4.2
- net at N1.3: now also J3.12 (Pin_12), N2.3, N3.3, N4.3
- net at N1.4: now also J3.13 (Pin_13), N2.4, N3.4, N4.4
- net at N1.5: now also J3.14 (Pin_14), N2.5, N3.5, N4.5
- net at N1.6: now also J3.15 (Pin_15), N2.6, N3.6, N4.6
- net at N1.7: now also J3.16 (Pin_16), N2.7, N3.7, N4.7
- net at N1.8: now also J3.17 (Pin_17), N2.8, N3.8, N4.8
- net at N1.9: now also J3.18 (Pin_18), N2.9, N3.9, N4.9
- net at N1.A: now also J3.6 (Pin_6)
- new net: LED1.1, Q1.6 (C1)
- new net: J3.3 (Pin_3), N4.A
- new net: J3.4 (Pin_4), N3.A
- new net: J3.5 (Pin_5), N2.A
- new net: LED2.1, Q1.3 (C2)
- new net: LED3.1, Q2.6 (C1)
- new net: LED4.1, Q2.3 (C2)
- new net: Q1.2 (B1), Q1.5 (B2), Q2.2 (B1), Q2.5 (B2), RV1.2
- new net: Q1.1 (E1), RA9.8 (R1.2)
- new net: Q2.1 (E1), RA9.6 (R3.2)
- new net: Q1.4 (E2), RA9.7 (R2.2)
- new net: Q2.4 (E2), RA9.5 (R4.2)
- new net +3V0: J3.20 (Pin_20), RV1.1
- new net GND: J3.1 (Pin_1), J3.19 (Pin_19), RA9.1 (R1.1), RA9.2 (R2.1), RA9.3 (R3.1), RA9.4 (R4.1), RV1.3
- new net VCC: J3.2 (Pin_2), LED1.2, LED2.2, LED3.2, LED4.2
- new net colon1: GL1.1 (A), J3.7 (Pin_7)
- new net colon2: GL1.2 (A1), J3.8 (Pin_8)
- no-connect marks 0 -> 8
Other:
- moved on the sheet: N1

Commit message: PCB as submitted to fab
Parts:
- GL1: value NE2-NEON-BULB-DRILL -> A1A; footprint mynixies:mynixies-NE2-NEON-BULB-DRILL -> footprints:NE2-A1A; symbol mynixies:NE2-NEON-BULB-DRILL -> ne2-a1a:NE2-A1A
- N1, N2, N3, N4: footprint nixies-us:nixies-us-IN-14 -> footprints:IN-14; symbol nixies-us:IN-14 -> in14:IN-14
Connections:
- net labels added: HR1, HR10, MIN1, MIN10
- wire segments 100 -> 75
- no-connect marks 8 -> 0
Other:
- moved on the sheet: J3, LED1, LED2, LED3, LED4, Q1A, Q1B, Q2A, Q2B, RA9, RV1
