File: Hardware/socket/in14-socket/in14-socket.kicad_pcb (KiCad board)
At the start: 2 copper layers, 14 parts, among them J3 Conn_01x20_Male, Q1 BC847BS, Q2 BC847BS

Commit message: PCB as submitted to fab
Parts:
- added H1: MountingHole_2.7mm_M2.5, MountingHole:MountingHole_2.7mm_M2.5, F.Cu at (127.0, 108.0)
- added H2: MountingHole_2.7mm_M2.5, MountingHole:MountingHole_2.7mm_M2.5, F.Cu at (127.0, 93.0)
- added H3: MountingHole_2.7mm_M2.5, MountingHole:MountingHole_2.7mm_M2.5, F.Cu at (193.0, 93.0)
- added H4: MountingHole_2.7mm_M2.5, MountingHole:MountingHole_2.7mm_M2.5, F.Cu at (193.0, 108.0)
- added H5: MountingHole_2.7mm_M2.5, MountingHole:MountingHole_2.7mm_M2.5, F.Cu at (160.0, 108.0)
- GL1: value NE2-NEON-BULB-DRILL -> A1A; footprint mynixies:mynixies-NE2-NEON-BULB-DRILL -> footprints:NE2-A1A
- N1, N2, N3, N4: footprint nixies-us:nixies-us-IN-14 -> footprints:IN-14
- Q1, Q2, RA9: moved to B.Cu
- moved LED1 77.6 mm to (204.5, 99.0)
- moved N1 77.6 mm to (204.5, 99.0)
- moved Q1 63.4 mm to (183.0, 115.0), turned to 270 degrees
- moved LED2 49.1 mm to (181.5, 99.0)
- moved N2 49.0 mm to (181.5, 99.0)
- moved RA9 47.6 mm to (160.0, 116.0), turned to 90 degrees
- moved N4 41.4 mm to (115.5, 99.0)
- moved LED4 41.4 mm to (115.5, 99.0)
- moved N3 37.7 mm to (138.5, 99.0)
- moved LED3 37.7 mm to (138.5, 99.0)
- moved J3 36.4 mm to (160.0, 130.0), turned to 180 degrees
- moved GL1 36.2 mm to (160.0, 99.0), turned to 90 degrees
- moved Q2 25.5 mm to (136.0, 115.0), turned to 90 degrees
- moved RV1 25.0 mm to (131.0, 123.0)
Connections:
- net Net-(J3-Pad3) renamed /MIN1
- net Net-(J3-Pad4) renamed /MIN10
- net Net-(J3-Pad5) renamed /HR1
- net Net-(J3-Pad6) renamed /HR10
Routing:
- net Net-(J3-Pad18): track 0.00 -> 159.7 mm
- net Net-(J3-Pad9): track 0.00 -> 142.9 mm
- net Net-(J3-Pad14): track 0.00 -> 139.3 mm, vias 0 -> 1
- net VCC: track 0.00 -> 138.9 mm, vias 0 -> 1
- net Net-(J3-Pad16): track 0.00 -> 138.0 mm, vias 0 -> 1
- net Net-(J3-Pad15): track 0.00 -> 135.1 mm
- net Net-(J3-Pad13): track 0.00 -> 132.6 mm, vias 0 -> 1
- net Net-(J3-Pad17): track 0.00 -> 132.4 mm
- net Net-(J3-Pad11): track 0.00 -> 130.8 mm, vias 0 -> 1
- net Net-(J3-Pad10): track 0.00 -> 128.0 mm
- net Net-(J3-Pad12): track 0.00 -> 126.4 mm
- net Net-(Q1-Pad2): track 0.00 -> 66.2 mm, vias 0 -> 1
- net /MIN1: track 0.00 -> 62.6 mm
- net Net-(Q2-Pad1): track 0.00 -> 56.9 mm
- net /HR10: track 0.00 -> 50.2 mm
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Other:
- board outline added: 105 x 40 mm

Commit message: fix switch pin assignment, reduce hole size on nixie sockets
Parts:
- N1, N2, N3, N4: value IN-14 -> Val**

Commit message: relocate libraries for socket boards, fix routing & 3D models
Routing:
- net GND: track 37.1 -> 68.2 mm, vias 0 -> 1
Changed lines of the file:
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@@
     (thickness 1.6)
     (drawings 9)
-    (tracks 398)
+    (tracks 403)
     (zones 0)
     (modules 19)
@@
     (0 F.Cu signal)
     (31 B.Cu signal)
-    (32 B.Adhes user)
-    (33 F.Adhes user)
+    (32 B.Adhes user hide)
+    (33 F.Adhes user hide)
     (34 B.Paste user)
     (35 F.Paste user)
-    (36 B.SilkS user)
+    (36 B.SilkS user hide)
     (37 F.SilkS user)
     (38 B.Mask user)
-    (39 F.Mask user)
+    (39 F.Mask user hide)
     (40 Dwgs.User user hide)
     (41 Cmts.User user)
@@
       (effects (font (size 1.27 1.27) (thickness 0.1016)))
     )
-    (fp_text value Val** (at 0 0) (layer F.SilkS)
+    (fp_text value Val** (at 0 0) (layer Cmts.User)
       (effects (font (size 1.27 1.27) (thickness 0.15)))
     )
@@
       (effects (font (size 1.27 1.27) (thickness 0.1016)))
     )
-    (fp_text value Val** (at 0 0) (layer F.SilkS)
+    (fp_text value Val** (at 0 0) (layer Cmts.User)
       (effects (font (size 1.27 1.27) (thickness 0.15)))
     )
@@
       (effects (font (size 1.27 1.27) (thickness 0.1016)))
     )
-    (fp_text value Val** (at 0 0) (layer F.SilkS)
+    (fp_text value Val** (at 0 0) (layer Cmts.User)
       (effects (font (size 1.27 1.27) (thickness 0.15)))
     )
@@
       (effects (font (size 1.27 1.27) (thickness 0.1016)))
     )
-    (fp_text value Val** (at 0 0) (layer F.SilkS)
+    (fp_text value Val** (at 0 0) (layer Cmts.User)
       (effects (font (size 1.27 1.27) (thickness 0.15)))
     )
@@
     (pad 3 thru_hole circle (at 2.54 0 90) (size 1.222 1.222) (drill 0.714) (layers *.Cu *.Mask)
       (net 10 GND))
+    (model ${KISYS3DMOD}/Potentiometer_THT.3dshapes/Potentiometer_Bourns_3339H_Vertical.wrl
+      (offset (xyz 2.5 0 0))
+      (scale (xyz 1.3 1.4 0.8))
+      (rotate (xyz 0 0 -90))
+    )
   )
   (module Resistor_SMD:R_Array_Convex_4x0603 (layer B.Cu)
@@
   (segment (start 159.6 116.9) (end 160.4 116.9) (width 0.25) (layer B.Cu) (net 10))
   (segment (start 160.4 116.9) (end 161.2 116.9) (width 0.25) (layer B.Cu) (net 10))
+  (via (at 159.9 117.978) (size 0.8) (drill 0.4) (layers F.Cu B.Cu) (net 10))
+  (segment (start 159.6 117.678) (end 159.9 117.978) (width 0.25) (layer B.Cu) (net 10))
+  (segment (start 159.6 116.9) (end 159.6 117.678) (width 0.25) (layer B.Cu) (net 10))
+  (segment (start 157.418 120.46) (end 131 120.46) (width 0.25) (layer F.Cu) (net 10))
+  (segment (start 159.9 117.978) (end 157.418 120.46) (width 0.25) (layer F.Cu) (net 10))
   (segment (start 134.3418 99.8655) (end 132.9821 101.2252) (width 0.25) (layer B.Cu) (net 11))
   (segment (start 132.9821 101.2252) (end 114.1337 101.2252) (width 0.25) (layer B.Cu) (net 11))

Commit message: fix routing on in-14 socket, make figures
Routing:
- net /colon1: track 30.1 -> 38.6 mm
- net Net-(J3-Pad15): track 135.1 -> 142.2 mm, vias 0 -> 1
- net Net-(J3-Pad14): track 139.3 -> 144.2 mm
- net Net-(J3-Pad13): track 132.6 -> 136.1 mm
- net Net-(J3-Pad16): track 138.0 -> 141.5 mm
